File: EAGLE Board Designs/Filter Board/playgroundFilter.sch (EAGLE design)
At the start: 9 parts, among them U1 MAX7400

Commit message: Prototype filter schematic
my eagle is scuffed :(
Parts:
- added C25, C27, C29, C31, C33, C35, C37, C39, C41, C43, C45, C47: CAPACITOR_0603_10V_0.1UF, HyTechDevices:CAPACITOR_0603_10V_0.1UF
- added C26, C30, C34, C38, C42, C46: CAPACITOR_0603_10V_1UF, HyTechDevices:CAPACITOR_0603_10V_1UF
- added C28, C32, C36, C40, C44, C48: CAPACITOR_0603_10V_680PF, HyTechDevices:CAPACITOR_0603_10V_680PF
- added U10, U11, U6, U7, U8, U9: MAX7400, HyTechDevices:MAX7400
Connections:
- net INPUT_SIGNAL renamed N$1
- net OUTPUT_SIGNAL renamed N$2
- net RAW_24V_SIGNAL renamed N$5
- new net N$13: C28.1, U6.CLK
- new net N$14: C27.1, U6.COM, U6.OS
- new net N$15: C32.1, U7.CLK
- new net N$16: C31.1, U7.COM, U7.OS
- new net N$17: C36.1, U8.CLK
- new net N$18: C35.1, U8.COM, U8.OS
- new net N$19: C40.1, U9.CLK
- new net N$20: C39.1, U9.COM, U9.OS
- new net N$21: C44.1, U10.CLK
- new net N$22: C43.1, U10.COM, U10.OS
- new net N$23: C48.1, U11.CLK
- new net N$24: C47.1, U11.COM, U11.OS
- new net SPN_POT_1: U6.OUT
- new net SPN_POT_1_EXT_5V: U6.IN
- new net SPN_POT_2: U7.OUT
- new net SPN_POT_2_EXT_5V: U7.IN
- new net SPN_POT_3: U8.OUT
- new net SPN_POT_3_EXT_5V: U8.IN
- new net SPN_POT_4: U9.OUT
- new net SPN_POT_4_EXT_5V: U9.IN
- new net SPN_POT_5: U10.OUT
- new net SPN_POT_5_EXT_5V: U10.IN
- new net SPN_POT_6: U11.OUT
- new net SPN_POT_6_EXT_5V: U11.IN
- net +5V: now also U10.!SHDN, U10.VDD, U11.!SHDN, U11.VDD, U6.!SHDN, U6.VDD, U7.!SHDN, U7.VDD, U8.!SHDN, U8.VDD, U9.!SHDN, U9.VDD
- net GND: now also C25.2, C26.2, C27.2, C28.2, C29.2, C30.2, C31.2, C32.2, C33.2, C34.2, C35.2, C36.2, C37.2, C38.2, C39.2, C40.2, C41.2, C42.2, C43.2, C44.2, C45.2, C46.2, C47.2, C48.2, U10.GND, U11.GND, U6.GND, U7.GND, U8.GND, U9.GND
- net REGULATED_FREQ: now also C25.1, C26.1, C29.1, C30.1, C33.1, C34.1, C37.1, C38.1, C41.1, C42.1, C45.1, C46.1
Other:
- moved on the sheet: R2, R3
