File: EAGLE Board Designs/Filter Board/Filter Board rev1.brd (EAGLE design)
At the start: 76.2 x 152.4 mm, 122 parts, among them J4 CONNECTOR-40__, J5 CONNECTOR-40__, U10 MAX7400, U11 MAX7400, U19 MAX7400, U20 MAX7400, U21 MAX7400, U22 MAX7400, U23 MAX7400, U24 MAX7400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

Commit message: Update Filter Board
Parts:
- moved U11 7.28 mm to (19.1, 35.1)
- moved C46 7.28 mm to (14.0, 32.3)
- moved C45 7.28 mm to (11.7, 32.3)
- moved C48 7.28 mm to (24.9, 37.1)
- moved R41 7.28 mm to (14.0, 36.6)
- moved R42 7.28 mm to (12.2, 36.6)
- moved C47 7.28 mm to (24.9, 34.3)
- moved U24 4.58 mm to (35.6, 32.3)
- moved C103 4.58 mm to (41.4, 31.5)
- moved C104 4.58 mm to (41.4, 34.3)
- moved R44 4.58 mm to (28.7, 33.8)
- moved C101 4.58 mm to (28.2, 29.5)
- moved C102 4.58 mm to (30.5, 29.5)
- moved R43 4.58 mm to (30.5, 33.8)
- moved C3 4.34 mm to (59.2, 39.4)
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Routing:
- net CURRENT: track 0.00 -> 82.4 mm
- net CURRENT_EXT: track 0.00 -> 66.6 mm, vias 0 -> 2
- net REFERENCE_EXT: track 0.00 -> 50.2 mm, vias 0 -> 2
- net REFERENCE: track 0.00 -> 49.5 mm
- net BRAKE_PRESSURE_F: track 2.07 -> 24.8 mm, vias 0 -> 2
- net BRAKE_PRESSURE_R: track 1.82 -> 16.5 mm, vias 0 -> 2
- net BRAKE_PRESSURE_R_EXT: track 11.6 -> 15.0 mm
- net BRAKE_PRESSURE_F_EXT: track 18.4 -> 21.2 mm

Commit message: Next Step: Compact
Parts:
- moved C102 17.0 mm to (13.7, 32.0)
- moved R43 17.0 mm to (13.7, 36.3)
- moved R44 17.0 mm to (11.9, 36.3)
- moved U24 17.0 mm to (18.8, 34.8)
- moved C101 17.0 mm to (11.4, 32.0)
- moved C103 17.0 mm to (24.6, 34.0)
- moved C104 17.0 mm to (24.6, 36.8)
- moved C47 16.7 mm to (41.4, 32.0)
- moved C48 16.7 mm to (41.4, 34.8)
- moved R42 16.7 mm to (28.7, 34.3)
- moved U11 16.7 mm to (35.6, 32.8)
- moved C45 16.7 mm to (28.2, 30.0)
- moved C46 16.7 mm to (30.5, 30.0)
- moved R41 16.7 mm to (30.5, 34.3)
- moved C51 7.15 mm to (34.0, 82.8)
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Routing:
- net CURRENT: track 82.4 -> 35.2 mm
- net REFERENCE_EXT: track 50.2 -> 87.7 mm, vias 2 -> 1
- net CURRENT_EXT: track 66.6 -> 42.7 mm, vias 2 -> 1
- net +5V: track 75.3 -> 94.4 mm
- net SPN_POT_6_EXT: track 72.1 -> 58.0 mm
- net SPN_POT_6: track 89.5 -> 78.3 mm
- net BRAKE_PRESSURE_R: track 16.5 -> 10.4 mm, vias 2 -> 1
- net BRAKE_PRESSURE_F: track 24.8 -> 18.7 mm, vias 2 -> 1
- net REFERENCE: track 49.5 -> 53.8 mm

Commit message: compact filter
Parts:
- moved C101 39.8 mm to (51.1, 27.9)
- moved C102 39.8 mm to (53.3, 27.9)
- moved R43 39.8 mm to (53.3, 32.3)
- moved U24 39.8 mm to (58.4, 30.7)
- moved C103 39.8 mm to (64.3, 30.0)
- moved C104 39.8 mm to (64.3, 32.8)
- moved R44 39.8 mm to (51.6, 32.3)
- moved R10 31.7 mm to (41.1, 100.3)
- moved R9 31.7 mm to (42.9, 100.3)
- moved C1 31.7 mm to (49.5, 97.8)
- moved C52 31.7 mm to (46.2, 97.8)
- moved R1 31.7 mm to (49.5, 99.6)
- moved R22 31.7 mm to (46.2, 99.6)
- moved R6 30.5 mm to (53.6, 98.3)
- moved C53 30.5 mm to (58.7, 95.8)
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Routing:
- net REFERENCE_EXT: track 87.7 -> 18.9 mm, vias 1 -> 0
- net SPN_POT_6: track 78.3 -> 16.6 mm
- net SPN_POT_6_EXT: track 58.0 -> 13.7 mm
- net REFERENCE: track 53.8 -> 11.4 mm
- net SPN_POT_1: track 56.0 -> 19.8 mm
- net SPN_POT_1_EXT: track 61.4 -> 27.0 mm
- net SPN_POT_2_EXT: track 46.3 -> 13.8 mm
- net SPN_POT_2: track 40.5 -> 7.98 mm
- net ACCEL_1: track 55.8 -> 26.6 mm
- net BRAKE_2_EXT: track 50.7 -> 21.9 mm
- net BRAKE_1: track 56.7 -> 28.4 mm
- net ACCEL_2: track 36.8 -> 10.4 mm
- net STEERING_1: track 53.6 -> 29.0 mm
- net ACCEL_2_EXT: track 49.6 -> 25.1 mm
- net LOAD_FL: track 55.0 -> 31.6 mm
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
Commit message: more!
Parts:
- moved C101 1.02 mm to (51.1, 29.0)
- moved C102 1.02 mm to (53.3, 29.0)
- moved C103 1.02 mm to (64.3, 31.0)
- moved C104 1.02 mm to (64.3, 33.8)
- moved R43 1.02 mm to (53.3, 33.3)
- moved R44 1.02 mm to (51.6, 33.3)
- moved U24 1.02 mm to (58.4, 31.8)
Routing:
- net BRAKE_PRESSURE_R_EXT: track 11.7 -> 11.1 mm

Commit message: I'll take another look tomorrow
Improved filter and wire alignment
Parts:
- moved C33 30.0 mm to (5.59, 66.3)
- moved C35 30.0 mm to (18.8, 68.3)
- moved C36 30.0 mm to (18.8, 71.1)
- moved U8 30.0 mm to (13.0, 69.1)
- moved C34 30.0 mm to (7.87, 66.3)
- moved C45 27.7 mm to (5.33, 30.2)
- moved U11 27.7 mm to (12.7, 33.0)
- moved C47 27.7 mm to (18.5, 32.3)
- moved C48 27.7 mm to (18.5, 35.1)
- moved R42 27.7 mm to (5.84, 34.5)
- moved C46 27.7 mm to (7.62, 30.2)
- moved R41 27.7 mm to (7.62, 34.5)
- moved C97 27.4 mm to (5.33, 39.4)
- moved C98 27.4 mm to (7.62, 39.4)
- moved U23 27.4 mm to (12.7, 42.2)
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Routing:
- net ACCEL_1: track 26.6 -> 31.4 mm
- net ACCEL_1_EXT: track 40.4 -> 44.0 mm
- net CURRENT_EXT: track 37.8 -> 40.3 mm
- net SPN_POT_3: track 22.8 -> 20.5 mm
- net STEERING_2_EXT: track 38.7 -> 40.9 mm
- net LOAD_FL_EXT: track 41.0 -> 38.9 mm
- net SPN_POT_5: track 24.1 -> 21.9 mm
- net LOAD_FL: track 31.6 -> 33.6 mm
- net STEERING_2: track 31.8 -> 33.7 mm
- net REFERENCE_EXT: track 19.3 -> 21.1 mm
- net CURRENT: track 33.5 -> 35.2 mm
- net SPN_POT_5_EXT: track 30.5 -> 28.8 mm
- net REFERENCE: track 10.9 -> 12.5 mm
- net LOAD_RR: track 33.3 -> 31.8 mm
- net SPN_POT_1: track 19.8 -> 21.2 mm
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Other:
- board size 76.2 x 152.4 mm -> 50.8 x 152.4 mm

Commit message: Large Logo for Large Frequencies
to be filtered later...
Parts:
- added U$5: (no value), HyTechManufacturing:LOGO_HYTECH_LARGE
- moved C28 2.81 mm to (36.1, 110.7)
- moved C27 2.81 mm to (36.1, 108.0)
- moved U6 2.81 mm to (30.2, 108.7)
- moved C25 2.81 mm to (22.9, 105.9)
- moved C26 2.81 mm to (25.1, 105.9)
- moved R27 2.81 mm to (25.1, 110.2)
- moved R28 2.81 mm to (23.4, 110.2)
- moved C41 0.76 mm to (23.1, 114.3)
- moved C43 0.76 mm to (36.3, 116.3)
- moved C44 0.76 mm to (36.3, 119.1)
- moved R40 0.76 mm to (23.6, 118.6)
- moved U10 0.76 mm to (30.5, 117.1)
- moved C42 0.76 mm to (25.4, 114.3)
- moved R39 0.76 mm to (25.4, 118.6)
Routing:
- net LOAD_FR_EXT: track 23.5 -> 20.5 mm
- net LOAD_RL: track 9.35 -> 12.2 mm
- net LOAD_RL_EXT: track 17.3 -> 19.4 mm
- net LOAD_FR: track 11.7 -> 10.9 mm
Other:
- board text added: "HyTech Racing 2023 Filter Board rev1 Designed by Eric Galluzzi"

Commit message: quick fix
Connections:
- net GND: now also C45.2
Changed lines of the file:
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@@
 <vertex x="51.054" y="152.654"/>
 </polygon>
+<contactref element="C45" pad="2"/>
 <wire x1="45.45" y1="119.87" x2="45.45" y2="121.87" width="0" layer="19" extent="1-1"/>
 <wire x1="45.45" y1="117.87" x2="45.45" y2="119.87" width="0" layer="19" extent="1-1"/>
@@
 <wire x1="45.45" y1="87.87" x2="45.45" y2="89.87" width="0" layer="19" extent="1-1"/>
 <wire x1="45.45" y1="85.87" x2="45.45" y2="87.87" width="0" layer="19" extent="1-1"/>
-<wire x1="36.818" y1="107.95" x2="45.45" y2="107.87" width="0" layer="19" extent="1-1"/>
-<wire x1="36.818" y1="110.744" x2="36.818" y2="107.95" width="0" layer="19" extent="1-1"/>
-<wire x1="37.072" y1="116.332" x2="36.818" y2="110.744" width="0" layer="19" extent="1-1"/>
+<wire x1="37.072" y1="116.332" x2="45.45" y2="115.87" width="0" layer="19" extent="1-1"/>
 <wire x1="37.072" y1="119.126" x2="37.072" y2="116.332" width="0" layer="19" extent="1-1"/>
+<wire x1="36.818" y1="110.744" x2="37.072" y2="116.332" width="0" layer="19" extent="1-1"/>
+<wire x1="36.818" y1="107.95" x2="36.818" y2="110.744" width="0" layer="19" extent="1-1"/>
 <wire x1="27.8765" y1="116.459" x2="37.072" y2="116.332" width="0" layer="19" extent="1-1"/>
 <wire x1="25.4" y1="113.55" x2="27.8765" y2="116.459" width="0" layer="19" extent="1-1"/>
 <wire x1="23.114" y1="113.55" x2="25.4" y2="113.55" width="0" layer="19" extent="1-1"/>
-<wire x1="23.368" y1="111.086" x2="25.4" y2="113.55" width="0" layer="19" extent="1-1"/>
+<wire x1="23.368" y1="111.086" x2="23.114" y2="113.55" width="0" layer="19" extent="1-1"/>
 <wire x1="19.546" y1="112.268" x2="23.114" y2="113.55" width="0" layer="19" extent="1-1"/>
 <wire x1="19.546" y1="109.474" x2="19.546" y2="112.268" width="0" layer="19" extent="1-1"/>
@@
 <wire x1="10.0965" y1="32.385" x2="7.62" y2="38.62" width="0" layer="19" extent="1-1"/>
 <wire x1="7.62" y1="29.476" x2="10.0965" y2="32.385" width="0" layer="19" extent="1-1"/>
+<wire x1="5.334" y1="29.476" x2="7.62" y2="29.476" width="0" layer="19" extent="1-1"/>
 </signal>
 <signal name="LOAD_FL_EXT">

Commit message: inverted design
Parts:
- added U$6: (no value), HyTechManufacturing:LOGO_HYTECH_LARGE
Connections:
- removed net GND1: R12.2, R16.2
- removed net GND2: R14.2, R18.2, R42.2, R44.2
- net GND: now also R12.2, R14.2, R16.2, R18.2, R44.2
Routing:
- net SPN_POT_4: track 6.35 -> 8.03 mm
