File: EAGLE Board Designs/Filter Board/Filter Board rev1.brd (EAGLE design)
At the start: 50.8 x 152.4 mm, 124 parts, among them J4 CONNECTOR-40__, J5 CONNECTOR-40__, U10 MAX7400, U11 MAX7400, U19 MAX7400, U20 MAX7400, U21 MAX7400, U22 MAX7400, U23 MAX7400, U24 MAX7400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

Commit message: GOt it
Routing:
- net BRAKE_1_EXT: track 44.5 -> 43.6 mm
- net STEERING_2: track 33.7 -> 33.0 mm
- net REFERENCE_EXT: track 21.1 -> 20.5 mm
- net STEERING_1_EXT: track 46.3 -> 45.7 mm
Changed lines of the file:
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@@
 <drawing>
 <settings>
-<setting alwaysvectorfont="no"/>
+<setting alwaysvectorfont="yes"/>
 <setting verticaltext="up"/>
 </settings>
@@
 <wire x1="7.874" y1="62.484" x2="9.652" y2="64.262" width="0.254" layer="1"/>
 <wire x1="19.558" y1="64.262" x2="20.828" y2="62.992" width="0.254" layer="1"/>
-<wire x1="20.828" y1="62.992" x2="20.828" y2="59.69" width="0.254" layer="1"/>
-<wire x1="20.828" y1="59.69" x2="21.48" y2="59.038" width="0.254" layer="1"/>
-<wire x1="42.942" y1="59.038" x2="43.45" y2="58.53" width="0.254" layer="1"/>
-<wire x1="42.942" y1="59.038" x2="21.48" y2="59.038" width="0.254" layer="1"/>
+<wire x1="20.828" y1="62.992" x2="20.828" y2="61.214" width="0.254" layer="1"/>
+<wire x1="20.828" y1="61.214" x2="22.75" y2="59.292" width="0.254" layer="1"/>
+<wire x1="42.688" y1="59.292" x2="43.45" y2="58.53" width="0.254" layer="1"/>
+<wire x1="42.688" y1="59.292" x2="22.75" y2="59.292" width="0.254" layer="1"/>
 <wire x1="9.652" y1="64.262" x2="19.558" y2="64.262" width="0.254" layer="1"/>
 </signal>
@@
 <wire x1="27.559" y1="53.721" x2="26.67" y2="54.61" width="0.254" layer="1"/>
 <wire x1="26.67" y1="54.61" x2="26.67" y2="56.134" width="0.254" layer="1"/>
-<wire x1="26.67" y1="56.134" x2="27.686" y2="57.15" width="0.254" layer="1"/>
-<wire x1="27.686" y1="57.15" x2="40.83" y2="57.15" width="0.254" layer="1"/>
-<wire x1="40.83" y1="57.15" x2="43.45" y2="54.53" width="0.254" layer="1"/>
+<wire x1="26.67" y1="56.134" x2="27.432" y2="56.896" width="0.254" layer="1"/>
+<wire x1="27.432" y1="56.896" x2="41.084" y2="56.896" width="0.254" layer="1"/>
+<wire x1="41.084" y1="56.896" x2="43.45" y2="54.53" width="0.254" layer="1"/>
 </signal>
 <signal name="BRAKE_PRESSURE_F_EXT">
@@
 <wire x1="9.652" y1="55.626" x2="19.05" y2="55.626" width="0.254" layer="1"/>
 <wire x1="19.05" y1="55.626" x2="21.082" y2="53.594" width="0.254" layer="1"/>
-<wire x1="21.082" y1="53.594" x2="21.082" y2="49.53" width="0.254" layer="1"/>
-<wire x1="21.082" y1="49.53" x2="22.098" y2="48.514" width="0.254" layer="1"/>
+<wire x1="21.082" y1="53.594" x2="21.082" y2="50.546" width="0.254" layer="1"/>
+<wire x1="21.082" y1="50.546" x2="23.114" y2="48.514" width="0.254" layer="1"/>
 <wire x1="41.434" y1="48.514" x2="43.45" y2="50.53" width="0.254" layer="1"/>
 <wire x1="7.874" y1="53.848" x2="9.652" y2="55.626" width="0.254" layer="1"/>
-<wire x1="22.098" y1="48.514" x2="41.434" y2="48.514" width="0.254" layer="1"/>
+<wire x1="23.114" y1="48.514" x2="41.434" y2="48.514" width="0.254" layer="1"/>
 </signal>
 <signal name="STEERING_2_EXT">
@@
 <contactref element="R41" pad="1"/>
 <wire x1="7.62" y1="35.394" x2="7.62" y2="36.156" width="0.254" layer="1"/>
-<wire x1="40.77919375" y1="39.459" x2="44.34280625" y2="39.459" width="0.254" layer="1"/>
 <wire x1="45.27180625" y1="38.53" x2="45.45" y2="38.53" width="0.254" layer="1"/>
-<wire x1="44.34280625" y1="39.459" x2="45.27180625" y2="38.53" width="0.254" layer="1"/>
-<wire x1="7.62" y1="36.156" x2="9.564" y2="38.1" width="0.254" layer="1"/>
-<wire x1="9.564" y1="38.1" x2="39.42019375" y2="38.1" width="0.254" layer="1"/>
-<wire x1="39.42019375" y1="38.1" x2="40.77919375" y2="39.459" width="0.254" layer="1"/>
+<wire x1="45.27180625" y1="38.53" x2="44.34280625" y2="39.459" width="0.254" layer="1"/>
+<wire x1="7.62" y1="36.156" x2="10.072" y2="38.608" width="0.254" layer="1"/>
+<wire x1="10.072" y1="38.608" x2="39.92819375" y2="38.608" width="0.254" layer="1"/>
+<wire x1="40.77919375" y1="39.459" x2="39.92819375" y2="38.608" width="0.254" layer="1"/>
+<wire x1="44.34280625" y1="39.459" x2="44.17780625" y2="39.624" width="0.254" layer="1"/>
+<wire x1="40.94419375" y1="39.624" x2="40.77919375" y2="39.459" width="0.254" layer="1"/>
+<wire x1="44.17780625" y1="39.624" x2="40.94419375" y2="39.624" width="0.254" layer="1"/>
 </signal>
 <signal name="REFERENCE_EXT">
 <contactref element="J5" pad="36"/>
 <contactref element="R43" pad="1"/>
-<wire x1="44.379" y1="35.601" x2="45.45" y2="34.53" width="0.254" layer="1"/>
-<wire x1="40.01719375" y1="35.601" x2="44.379" y2="35.601" width="0.254" layer="1"/>
-<wire x1="26.416" y1="34.124" x2="29.122" y2="36.83" width="0.254" layer="1"/>
-<wire x1="29.122" y1="36.83" x2="38.78819375" y2="36.83" width="0.254" layer="1"/>
-<wire x1="38.78819375" y1="36.83" x2="40.01719375" y2="35.601" width="0.254" layer="1"/>
+<wire x1="26.416" y1="34.124" x2="28.36" y2="36.068" width="0.254" layer="1"/>
+<wire x1="28.36" y1="36.068" x2="39.55019375" y2="36.068" width="0.254" layer="1"/>
+<wire x1="40.05819375" y1="35.56" x2="44.45" y2="35.56" width="0.254" layer="1"/>
+<wire x1="44.45" y1="35.56" x2="45.45" y2="34.56" width="0.254" layer="1"/>
+<wire x1="45.45" y1="34.56" x2="45.45" y2="34.53" width="0.254" layer="1"/>
+<wire x1="39.55019375" y1="36.068" x2="40.05819375" y2="35.56" width="0.254" layer="1"/>
 </signal>
 <signal name="LOAD_FL">
@@
 <wire x1="43.404" y1="89.916" x2="43.45" y2="89.87" width="0.254" layer="1"/>
 <wire x1="38.696" y1="89.916" x2="43.404" y2="89.916" width="0.254" layer="1"/>
-<wire x1="37.58" y1="87.122" x2="37.58" y2="88.8" width="0.1524" layer="1"/>
-<wire x1="37.58" y1="88.8" x2="37.68" y2="88.9" width="0.1524" layer="1"/>
+<wire x1="37.58" y1="87.122" x2="37.58" y2="88.8" width="0.254" layer="1"/>
+<wire x1="37.58" y1="88.8" x2="37.68" y2="88.9" width="0.254" layer="1"/>
 </signal>
 <signal name="SPN_POT_5">
@@
 <contactref element="J5" pad="13"/>
 <contactref element="U19" pad="5"/>
-<wire x1="41.687" y1="58.293" x2="15.5575" y2="58.293" width="0.254" layer="1"/>
-<wire x1="15.3035" y1="58.039" x2="15.5575" y2="58.293" width="0.254" layer="1"/>
-<wire x1="41.687" y1="58.293" x2="43.45" y2="56.53" width="0.254" layer="1"/>
+<wire x1="41.941" y1="58.039" x2="15.3035" y2="58.039" width="0.254" layer="1"/>
+<wire x1="41.941" y1="58.039" x2="43.45" y2="56.53" width="0.254" layer="1"/>
 </signal>
 <signal name="BRAKE_2">
@@
 <contactref element="J5" pad="25"/>
 <contactref element="U23" pad="5"/>
-<wire x1="15.3035" y1="40.259" x2="23.749" y2="40.259" width="0.254" layer="1"/>
-<wire x1="23.749" y1="40.259" x2="24.384" y2="40.894" width="0.254" layer="1"/>
-<wire x1="24.384" y1="40.894" x2="24.384" y2="44.958" width="0.254" layer="1"/>
+<wire x1="15.3035" y1="40.259" x2="22.479" y2="40.259" width="0.254" layer="1"/>
+<wire x1="22.479" y1="40.259" x2="24.384" y2="42.164" width="0.254" layer="1"/>
+<wire x1="24.384" y1="42.164" x2="24.384" y2="44.958" width="0.254" layer="1"/>
 <wire x1="24.384" y1="44.958" x2="25.654" y2="46.228" width="0.254" layer="1"/>
 <wire x1="41.752" y1="46.228" x2="43.45" y2="44.53" width="0.254" layer="1"/>
@@
 <wire x1="20.955" y1="31.115" x2="22.098" y2="32.258" width="0.254" layer="1"/>
 <wire x1="22.098" y1="32.258" x2="22.098" y2="35.814" width="0.254" layer="1"/>
-<wire x1="45.27180625" y1="36.53" x2="45.45" y2="36.53" width="0.254" layer="1"/>
-<wire x1="44.34280625" y1="37.459" x2="45.27180625" y2="36.53" width="0.254" layer="1"/>
+<wire x1="45.45" y1="36.53" x2="45.45" y2="36.60580625" width="0.254" layer="1"/>
+<wire x1="45.45" y1="36.60580625" x2="44.59680625" y2="37.459" width="0.254" layer="1"/>
 <wire x1="22.098" y1="35.814" x2="23.743" y2="37.459" width="0.254" layer="1"/>
-<wire x1="23.743" y1="37.459" x2="44.34280625" y2="37.459" width="0.254" layer="1"/>
+<wire x1="23.743" y1="37.459" x2="44.59680625" y2="37.459" width="0.254" layer="1"/>
 </signal>
 <signal name="REFERENCE">
 <contactref element="J5" pad="38"/>
 <contactref element="U24" pad="5"/>
-<wire x1="44.379" y1="31.459" x2="45.45" y2="32.53" width="0.254" layer="1"/>
-<wire x1="43.06519375" y1="31.459" x2="44.379" y2="31.459" width="0.254" layer="1"/>
-<wire x1="34.0995" y1="29.845" x2="41.45119375" y2="29.845" width="0.254" layer="1"/>
-<wire x1="41.45119375" y1="29.845" x2="43.06519375" y2="31.459" width="0.254" layer="1"/>
+<wire x1="34.0995" y1="29.845" x2="41.402" y2="29.845" width="0.254" layer="1"/>
+<wire x1="41.402" y1="29.845" x2="41.45119375" y2="29.845" width="0.254" layer="1"/>
+<wire x1="41.402" y1="29.845" x2="43.053" y2="31.496" width="0.254" layer="1"/>
+<wire x1="43.053" y1="31.496" x2="44.704" y2="31.496" width="0.254" layer="1"/>
+<wire x1="44.704" y1="31.496" x2="45.45" y2="32.242" width="0.254" layer="1"/>
+<wire x1="45.45" y1="32.242" x2="45.45" y2="32.53" width="0.254" layer="1"/>
 </signal>
 <signal name="SPN_POT_2_EXT_5V">

Commit message: embarassing
Connections:
- net GND: now also R42.2
Changed lines of the file:
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@@
 <contactref element="R18" pad="2"/>
 <contactref element="R44" pad="2"/>
+<contactref element="R42" pad="2"/>
 </signal>
 <signal name="LOAD_FL_EXT">
@@
 <contactref element="R41" pad="1"/>
 <wire x1="7.62" y1="35.394" x2="7.62" y2="36.156" width="0.254" layer="1"/>
-<wire x1="45.27180625" y1="38.53" x2="45.45" y2="38.53" width="0.254" layer="1"/>
-<wire x1="45.27180625" y1="38.53" x2="44.34280625" y2="39.459" width="0.254" layer="1"/>
+<wire x1="45.01780625" y1="38.53" x2="45.45" y2="38.53" width="0.254" layer="1"/>
+<wire x1="45.01780625" y1="38.53" x2="44.00000625" y2="39.5478" width="0.254" layer="1"/>
 <wire x1="7.62" y1="36.156" x2="10.072" y2="38.608" width="0.254" layer="1"/>
 <wire x1="10.072" y1="38.608" x2="39.92819375" y2="38.608" width="0.254" layer="1"/>
-<wire x1="40.77919375" y1="39.459" x2="39.92819375" y2="38.608" width="0.254" layer="1"/>
-<wire x1="44.34280625" y1="39.459" x2="44.17780625" y2="39.624" width="0.254" layer="1"/>
-<wire x1="40.94419375" y1="39.624" x2="40.77919375" y2="39.459" width="0.254" layer="1"/>
-<wire x1="44.17780625" y1="39.624" x2="40.94419375" y2="39.624" width="0.254" layer="1"/>
+<wire x1="40.86799375" y1="39.5478" x2="39.92819375" y2="38.608" width="0.254" layer="1"/>
+<wire x1="44.00000625" y1="39.5478" x2="40.86799375" y2="39.5478" width="0.254" layer="1"/>
 </signal>
 <signal name="REFERENCE_EXT">
@@
 <contactref element="U24" pad="5"/>
 <wire x1="34.0995" y1="29.845" x2="41.402" y2="29.845" width="0.254" layer="1"/>
-<wire x1="41.402" y1="29.845" x2="41.45119375" y2="29.845" width="0.254" layer="1"/>
 <wire x1="41.402" y1="29.845" x2="43.053" y2="31.496" width="0.254" layer="1"/>
 <wire x1="43.053" y1="31.496" x2="44.704" y2="31.496" width="0.254" layer="1"/>

Commit message: Updated for HyTech Default DRC
Routing:
- net GND: track 0.00 -> 52.1 mm, vias 0 -> 12
- added copper zone on layer 16, net GND
