File: EAGLE Board Designs/Filter Board/Filter Board rev1.sch (EAGLE design)
At the start: 118 parts, among them J4 CONNECTOR-40__, J5 CONNECTOR-40__, U10 MAX7400, U11 MAX7400, U19 MAX7400, U20 MAX7400, U21 MAX7400, U22 MAX7400, U23 MAX7400, U24 MAX7400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

Commit message: vector -> proportional
Other:
- note added: "24 to 4.859 = .1912"
- moved on the sheet: C101, C102, C103, C104, C25, C26, C27, C28, R27, R28, R43, R44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
